File: ClockLogicBoard.kicad_pcb (KiCad board)
At the start: 2 copper layers, 24 parts, among them SW1 SW_Push, SW2 SW_SPDT, U1 NE555P, U2 NE555P, U3 NE555P, U4 74LS04, U5 74LS08, U6 74LS32

Commit message: prototype
Parts:
- removed C10: 0.1uF, Capacitor_THT:C_Radial_D10.0mm_H12.5mm_P5.00mm
- removed D1: BLUE, LED_THT:LED_D5.0mm
- removed U5: 74LS08, Package_DIP:DIP-14_W7.62mm
- removed U6: 74LS32, Package_DIP:DIP-14_W7.62mm
- added C7: 0.1uF, Capacitor_THT:C_Disc_D8.0mm_W2.5mm_P5.00mm, F.Cu at (154.5, 102.2)
- added J1: Barrel_Jack, Connector_BarrelJack:BarrelJack_Horizontal, F.Cu at (170.0, 91.2)
- added J2: Conn_01x05_Male, Connector_PinHeader_2.54mm:PinHeader_1x05_P2.54mm_Vertical, F.Cu at (151.9, 116.2)
- added LED1: BLUE, LED_THT:LED_D5.0mm, F.Cu at (144.0, 119.2)
- C1, C2, C3, C5: footprint Capacitor_THT:C_Radial_D10.0mm_H12.5mm_P5.00mm -> Capacitor_THT:C_Disc_D8.0mm_W2.5mm_P5.00mm
- C4: footprint Capacitor_THT:C_Radial_D10.0mm_H12.5mm_P5.00mm -> Capacitor_THT:CP_Radial_D4.0mm_P1.50mm
- C6: footprint Capacitor_THT:CP_Radial_D4.0mm_P2.00mm -> Capacitor_THT:C_Disc_D8.0mm_W2.5mm_P5.00mm
- R1, R2, R3, R4, R5, R6, R7: footprint Resistor_THT:R_Axial_DIN0204_L3.6mm_D1.6mm_P7.62mm_Horizontal -> Resistor_THT:R_Axial_DIN0204_L3.6mm_D1.6mm_P5.08mm_Horizontal
- RV1: footprint Resistor_THT:R_Axial_DIN0204_L3.6mm_D1.6mm_P2.54mm_Vertical -> Potentiometer_THT:Potentiometer_Bourns_3296W_Vertical
- SW2: footprint Button_Switch_THT:SW_CuK_OS102011MA1QN1_SPDT_Angled -> Button_Switch_THT:SW_E-Switch_EG1271_DPDT
- U4: value 74LS04 -> GAL16V8; footprint Package_DIP:DIP-14_W7.62mm -> Package_DIP:DIP-20_W7.62mm
- moved C6 52.5 mm to (154.5, 97.2)
- moved C2 49.0 mm to (164.5, 102.2)
- moved C5 43.1 mm to (144.5, 102.2)
- moved R1 32.6 mm to (130.5, 96.4)
- moved RV1 32.3 mm to (133.1, 105.7), turned to 90 degrees
- moved SW1 29.1 mm to (129.8, 116.0)
- moved U4 26.9 mm to (139.6, 113.0)
- moved R7 26.8 mm to (140.2, 120.7), turned to 90 degrees
- moved U1 26.1 mm to (130.2, 84.4)
- moved R2 23.7 mm to (130.4, 100.2)
- moved U2 23.7 mm to (141.2, 84.4)
- moved U3 21.7 mm to (152.2, 84.4)
- moved R6 17.8 mm to (154.5, 80.2)
- moved C3 13.8 mm to (144.5, 97.2)
- moved R4 13.5 mm to (138.5, 80.2), turned to 0 degrees
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Connections:
- C2 pad 1: Net-(C2-Pad1) -> VCC
- R4 pad 1: Net-(C3-Pad1) -> Net-(C6-Pad1)
- RV1 pad 1: Net-(C6-Pad1) -> Net-(C4-Pad1)
- U1 pad 2: Net-(C6-Pad1) -> Net-(C4-Pad1)
- U1 pad 5: Net-(C5-Pad1) -> Net-(C3-Pad1)
- U1 pad 6: Net-(C6-Pad1) -> Net-(C4-Pad1)
- U2 pad 5: Net-(C2-Pad1) -> Net-(C5-Pad1)
- U2 pad 6: Net-(C3-Pad1) -> Net-(C6-Pad1)
- U2 pad 7: Net-(C3-Pad1) -> Net-(C6-Pad1)
- U3 pad 5: Net-(C4-Pad1) -> Net-(C7-Pad1)
- U4 pad 1: Net-(U3-Pad3) -> Net-(U1-Pad3)
- U4 pad 10: (no net) -> GND
- U4 pad 11: (no net) -> unconnected-(U4-Pad11)
- U4 pad 12: (no net) -> unconnected-(U4-Pad12)
- U4 pad 13: (no net) -> unconnected-(U4-Pad13)
- U4 pad 14: (no net) -> unconnected-(U4-Pad14)
- U4 pad 2: Net-(U4-Pad2) -> Net-(U2-Pad3)
- U4 pad 3: HLT -> Net-(U3-Pad3)
- U4 pad 4: Net-(U4-Pad4) -> HLT
- U4 pad 5: CLK -> unconnected-(U4-Pad5)
- U4 pad 6: ~{CLK} -> unconnected-(U4-Pad6)
- U4 pad 7: (no net) -> unconnected-(U4-Pad7)
- U4 pad 8: (no net) -> unconnected-(U4-Pad8)
- U4 pad 9: (no net) -> unconnected-(U4-Pad9)
Routing:
- net GND: track 255.1 -> 0.00 mm, vias 2 -> 1
- net VCC: track 186.9 -> 127.8 mm, vias 4 -> 1
- net Net-(R5-Pad1): track 74.7 -> 36.2 mm
- net CLK: track 60.5 -> 23.8 mm, vias 2 -> 0
- net Net-(C2-Pad1): track 34.5 -> 0.00 mm
- net Net-(R2-Pad2): track 41.5 -> 9.96 mm
- net Net-(C3-Pad1): track 40.6 -> 9.76 mm
- net ~{CLK}: track 0.00 -> 29.8 mm
- net Net-(U5-Pad3): track 28.2 -> 0.00 mm, vias 2 -> 0
- net Net-(U4-Pad2): track 28.0 -> 0.00 mm
- net Net-(U4-Pad4): track 27.7 -> 0.00 mm, vias 1 -> 0
- net Net-(U5-Pad6): track 27.3 -> 0.00 mm, vias 1 -> 0
- net Net-(C6-Pad1): track 47.6 -> 25.7 mm, vias 1 -> 0
- net Net-(C5-Pad1): track 29.2 -> 12.0 mm
- net Net-(U3-Pad3): track 42.4 -> 27.7 mm
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- added copper zone on B.Cu, net GND
- added copper zone on F.Cu, net GND
Other:
- board outline added: 47 x 46 mm
- rule pad_to_mask_clearance: 0 -> 0.05
