File: ClockLogicBoard.kicad_sch (KiCad schematic)
At the start: 24 parts, among them SW1 SW_Push, SW2 SW_SPDT, U1 NE555P, U2 NE555P, U3 NE555P, U4 74LS04, U5 74LS08, U6 74LS32

Commit message: prototype
Parts:
- removed U4: 74LS04, Package_DIP:DIP-14_W7.62mm, symbol 74xx:74LS04
- removed U5: 74LS08, Package_DIP:DIP-14_W7.62mm, symbol 74xx:74LS08
- removed U6: 74LS32, Package_DIP:DIP-14_W7.62mm, symbol 74xx:74LS32
- added J1: Barrel_Jack, Connector_BarrelJack:BarrelJack_Horizontal, symbol Connector:Barrel_Jack
- added J2: Conn_01x05_Male, Connector_PinHeader_2.54mm:PinHeader_1x05_P2.54mm_Vertical, symbol Connector:Conn_01x05_Male
- added U4: GAL16V8, Package_DIP:DIP-20_W7.62mm, symbol Logic_Programmable:GAL16V8
- C1: footprint Capacitor_THT:C_Radial_D10.0mm_H12.5mm_P5.00mm -> Capacitor_THT:C_Disc_D8.0mm_W2.5mm_P5.00mm
- C2: renamed from C10; footprint Capacitor_THT:C_Radial_D10.0mm_H12.5mm_P5.00mm -> Capacitor_THT:C_Disc_D8.0mm_W2.5mm_P5.00mm
- C3: renamed from C5; footprint Capacitor_THT:C_Radial_D10.0mm_H12.5mm_P5.00mm -> Capacitor_THT:C_Disc_D8.0mm_W2.5mm_P5.00mm
- C4: renamed from C6; footprint Capacitor_THT:CP_Radial_D4.0mm_P2.00mm -> Capacitor_THT:CP_Radial_D4.0mm_P1.50mm
- C5: renamed from C2; footprint Capacitor_THT:C_Radial_D10.0mm_H12.5mm_P5.00mm -> Capacitor_THT:C_Disc_D8.0mm_W2.5mm_P5.00mm
- C6: renamed from C3; footprint Capacitor_THT:C_Radial_D10.0mm_H12.5mm_P5.00mm -> Capacitor_THT:C_Disc_D8.0mm_W2.5mm_P5.00mm
- C7: renamed from C4; footprint Capacitor_THT:C_Radial_D10.0mm_H12.5mm_P5.00mm -> Capacitor_THT:C_Disc_D8.0mm_W2.5mm_P5.00mm
- R1, R2, R3, R4, R5, R6, R7: footprint Resistor_THT:R_Axial_DIN0204_L3.6mm_D1.6mm_P7.62mm_Horizontal -> Resistor_THT:R_Axial_DIN0204_L3.6mm_D1.6mm_P5.08mm_Horizontal
- RV1: footprint Resistor_THT:R_Axial_DIN0204_L3.6mm_D1.6mm_P2.54mm_Vertical -> Potentiometer_THT:Potentiometer_Bourns_3296W_Vertical
- SW2: footprint Button_Switch_THT:SW_CuK_OS102011MA1QN1_SPDT_Angled -> Button_Switch_THT:SW_E-Switch_EG1271_DPDT
- renumbered D1 to LED1
Connections:
- net CLK: now also J2.2 (Pin_2), U4.18 (IO2)
- net GND: now also J1.2, J2.5 (Pin_5), U4.10 (GND)
- net HLT: now also J2.4 (Pin_4), U4.4 (I4)
- net VCC: now also J1.1, J2.1 (Pin_1), U4.20 (VCC)
- net ~{CLK}: now also J2.3 (Pin_3), U4.19 (IO1)
- net at U2.3 (Q): now also U4.2 (I2)
- net at U1.3 (Q): now also U4.1 (I1/CLK)
- net at U3.3 (Q): now also U4.3 (I3)
- no-connect marks 2 -> 14
Other:
- company: (none) -> Mush Labs
- title: (none) -> Clock Logic Board
- moved on the sheet: C1, C2, C3, C4, C5, C6, C7, LED1, R1, R2, R3, R4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
